Commit message: rope object initiation

File: isaacgymenvs/assets/mjcf/solid_rope/rope.urdf (robot description, URDF)
Before this commit: robot solid_rope, 2 links, 1 joints
Links:
- link rope_link: mass 0.5 -> 0.25; geometry collision cylinder length=1.0 radius=0.01; visual mesh filename=textured_objects/rope.obj scale=0.5 0.5 1.0
Joints:
- joint rope_base_joint: origin xyz=0 0 0.5 rpy=0 0 0 -> xyz=0 0 0 rpy=0 0 0
